File: ArduinoBoat/PCBs/TAFLab Boat/TAFLab Sensors.kicad_pcb (KiCad board)
At the start: 2 copper layers, 171.5 x 110.4 mm, 20 parts

Commit message: PCB edits
Parts:
- moved U2 0.10 mm to (104.0, 66.5)
Connections:
- U11 pad 1: Net-(U10-GND) -> Net-(U11-GND)
- U14 pad 3: Net-(U10-GND) -> Net-(U11-GND)
- U16 pad 3: Net-(U10-GND) -> Net-(U11-GND)
- U17 pad 3: Net-(U10-GND) -> Net-(U11-GND)
Changed lines of the file:
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@@
 	(net 104 "unconnected-(A1-PadA14)")
 	(net 105 "unconnected-(A1-PadA13)")
+	(net 106 "Net-(U11-GND)")
 	(footprint "TAFLab-Footprint-Library:XBeeBreakout"
 		(layer "F.Cu")
@@
 			)
 		)
+		(sheetname "Root")
+		(sheetfile "TAFLab Sensors.kicad_sch")
 		(attr smd)
 		(fp_rect
@@
 		)
 	)
-	(footprint "TAFLab-Footprint-Library:LIS3MDL_Magnometer"
-		(layer "F.Cu")
-		(at 104 66.6)
-		(property "Reference" "U2"
-			(at 0 -0.5 0)
-			(unlocked yes)
-			(layer "F.SilkS")
-			(hide yes)
-			(effects
-				(font
-					(size 1 1)
-					(thickness 0.1)
-				)
-			)
-		)
-		(property "Value" "~"
-			(at 0 1 0)
-			(unlocked yes)
-			(layer "F.Fab")
-			(hide yes)
-			(effects
-				(font
-					(size 1 1)
-					(thickness 0.15)
-				)
-			)
-		)
-		(property "Footprint" "TAFLab-Footprint-Library:LIS3MDL_Magnometer"
-			(at 0 0 0)
-			(unlocked yes)
-			(layer "F.Fab")
-			(hide yes)
-			(effects
-				(font
-					(size 1 1)
-					(thickness 0.15)
-				)
-			)
-		)
-		(property "Datasheet" ""
-			(at 0 0 0)
-			(unlocked yes)
-			(layer "F.Fab")
-			(hide yes)
-			(effects
-				(font
-					(size 1 1)
-					(thickness 0.15)
-				)
-			)
-		)
-		(property "Description" ""
-			(at 0 0 0)
-			(unlocked yes)
-			(layer "F.Fab")
-			(hide yes)
-			(effects
-				(font
-					(size 1 1)
-					(thickness 0.15)
-				)
-			)
-		)
-		(sheetname "Root")
-		(sheetfile "TAFLab Sensors.kicad_sch")
-		(attr smd)
-		(fp_rect
-			(start -2.5 -13)
-			(end 15.5 13)
-			(stroke
-				(width 0.1)
-				(type default)
-			)
-			(fill none)
-			(layer "F.SilkS")
-		)
-		(fp_text user "${REFERENCE}"
-			(at -5.5 6.2 0)
-			(unlocked yes)
-			(layer "F.Fab")
-			(hide yes)
-			(effects
-				(font
-					(size 1 1)
-					(thickness 0.15)
-				)
-			)
-		)
-		(pad "1" thru_hole oval
-			(at 0 -7)
-			(size 1.7272 1.7272)
-			(drill 1.016)
-			(layers "*.Cu" "*.Mask")
-			(remove_unused_layers no)
-			(net 20 "Net-(U10-Vin)")
-			(pinfunction "Vin")
-			(pintype "power_in")
-			(thermal_bridge_angle 45)
-		)
-		(pad "2" thru_hole oval
-			(at 0 -4.5)
-			(size 1.7272 1.7272)
-			(drill 1.016)
-			(layers "*.Cu" "*.Mask")
-			(remove_unused_layers no)
-			(net 84 "unconnected-(U2-3Vo-Pad2)")
-			(pinfunction "3Vo")
-			(pintype "power_in+no_connect")
-			(thermal_bridge_angle 45)
-		)
-		(pad "3" thru_hole oval
-			(at 0 -2)
-			(size 1.7272 1.7272)
-			(drill 1.016)
-			(layers "*.Cu" "*.Mask")
-			(remove_unused_layers no)
-			(net 103 "Net-(U10-GND)")
-			(pinfunction "GND")
-			(pintype "power_in")
-			(thermal_bridge_angle 45)
-		)
-		(pad "4" thru_hole oval
-			(at 0 0.5)
-			(size 1.7272 1.7272)
-			(drill 1.016)
-			(layers "*.Cu" "*.Mask")
-			(remove_unused_layers no)
-			(net 38 "Net-(U13-SCL)")
-			(pinfunction "SCL")
-			(pintype "bidirectional")
-			(thermal_bridge_angle 45)
-		)
-		(pad "5" thru_hole oval
-			(at 0 3)
-			(size 1.7272 1.7272)
-			(drill 1.016)
-			(layers "*.Cu" "*.Mask")
-			(remove_unused_layers no)
-			(net 66 "Net-(U13-SDA)")
-			(pinfunction "SDA")
-			(pintype "bidirectional")
-			(thermal_bridge_angle 45)
-		)
-		(pad "6" thru_hole oval
-			(at 0 5.5)
-			(size 1.7272 1.7272)
-			(drill 1.016)
-			(layers "*.Cu" "*.Mask")
-			(remove_unused_layers no)
-			(net 83 "unconnected-(U2-INT-Pad6)")
-			(pinfunction "INT")
-			(pintype "bidirectional+no_connect")
-			(thermal_bridge_angle 45)
-		)
-	)
 	(footprint "TAFLab-Footprint-Library:MPU6050_IMU_Accelerometer"
 		(layer "F.Cu")
@@
 			(layers "*.Cu" "*.Mask")
 			(remove_unused_layers no)
-			(net 103 "Net-(U10-GND)")
+			(net 106 "Net-(U11-GND)")
 			(pinfunction "GND")
 			(pintype "power_in")
@@
 			(layers "*.Cu" "*.Mask")
 			(remove_unused_layers no)
-			(net 103 "Net-(U10-GND)")
+			(net 106 "Net-(U11-GND)")
 			(pinfunction "GND")
 			(pintype "power_in")
@@
 			(layers "*.Cu" "*.Mask")
 			(remove_unused_layers no)
+			(net 106 "Net-(U11-GND)")
+			(pinfunction "GND")
+			(pintype "power_in")
+		)
+	)
+	(footprint "TAFLab-Footprint-Library:LIS3MDL_Magnometer"
+		(layer "F.Cu")
+		(at 104 66.5)
+		(property "Reference" "U2"
+			(at 0 -0.5 0)
+			(unlocked yes)
+			(layer "F.SilkS")
+			(effects
+				(font
+					(size 1 1)
+					(thickness 0.1)
+				)
+			)
+		)
+		(property "Value" "~"
+			(at 0 1 0)
+			(unlocked yes)
+			(layer "F.Fab")
+			(effects
+				(font
+					(size 1 1)
+					(thickness 0.15)
+				)
+			)
+		)
+		(property "Footprint" "TAFLab-Footprint-Library:LIS3MDL_Magnometer"
+			(at 0 0 0)
+			(unlocked yes)
+			(layer "F.Fab")
+			(hide yes)
+			(effects
+				(font
+					(size 1 1)
+					(thickness 0.15)
+				)
+			)
+		)
+		(property "Datasheet" ""
+			(at 0 0 0)
+			(unlocked yes)
+			(layer "F.Fab")
+			(hide yes)
+			(effects
+				(font
+					(size 1 1)
+					(thickness 0.15)
+				)
+			)
+		)
+		(property "Description" ""
+			(at 0 0 0)
+			(unlocked yes)
+			(layer "F.Fab")
+			(hide yes)
+			(effects
+				(font
+					(size 1 1)
+					(thickness 0.15)
+				)
+			)
+		)
+		(sheetname "Root")
+		(sheetfile "TAFLab Sensors.kicad_sch")
+		(attr smd)
+		(fp_rect
+			(start -2.5 -13)
+			(end 15.5 13)
+			(stroke
+				(width 0.1)
+				(type default)
+			)
+			(fill none)
+			(layer "F.SilkS")
+		)
+		(fp_text user "${REFERENCE}"
+			(at 0 2.5 0)
+			(unlocked yes)
+			(layer "F.Fab")
+			(effects
+				(font
+					(size 1 1)
+					(thickness 0.15)
+				)
+			)
+		)
+		(pad "1" thru_hole oval
+			(at 0 -7)
+			(size 1.7272 1.7272)
+			(drill 1.016)
+			(layers "*.Cu" "*.Mask")
+			(remove_unused_layers no)
+			(net 20 "Net-(U10-Vin)")
+			(pinfunction "Vin")
+			(pintype "power_in")
+			(thermal_bridge_angle 45)
+		)
+		(pad "2" thru_hole oval
+			(at 0 -4.5)
+			(size 1.7272 1.7272)
+			(drill 1.016)
+			(layers "*.Cu" "*.Mask")
+			(remove_unused_layers no)
+			(net 84 "unconnected-(U2-3Vo-Pad2)")
+			(pinfunction "3Vo")
+			(pintype "power_in+no_connect")
+			(thermal_bridge_angle 45)
+		)
+		(pad "3" thru_hole oval
+			(at 0 -2)
+			(size 1.7272 1.7272)
+			(drill 1.016)
+			(layers "*.Cu" "*.Mask")
+			(remove_unused_layers no)
 			(net 103 "Net-(U10-GND)")
 			(pinfunction "GND")
 			(pintype "power_in")
+			(thermal_bridge_angle 45)
+		)
+		(pad "4" thru_hole oval
+			(at 0 0.5)
+			(size 1.7272 1.7272)
+			(drill 1.016)
+			(layers "*.Cu" "*.Mask")
+			(remove_unused_layers no)
+			(net 38 "Net-(U13-SCL)")
+			(pinfunction "SCL")
+			(pintype "bidirectional")
+			(thermal_bridge_angle 45)
+		)
+		(pad "5" thru_hole oval
+			(at 0 3)
+			(size 1.7272 1.7272)
+			(drill 1.016)
+			(layers "*.Cu" "*.Mask")
+			(remove_unused_layers no)
+			(net 66 "Net-(U13-SDA)")
+			(pinfunction "SDA")
+			(pintype "bidirectional")
+			(thermal_bridge_angle 45)
+		)
+		(pad "6" thru_hole oval
+			(at 0 5.5)
+			(size 1.7272 1.7272)
+			(drill 1.016)
+			(layers "*.Cu" "*.Mask")
+			(remove_unused_layers no)
+			(net 83 "unconnected-(U2-INT-Pad6)")
+			(pinfunction "INT")
+			(pintype "bidirectional+no_connect")
+			(thermal_bridge_angle 45)
 		)
 	)
@@
 			(layers "*.Cu" "*.Mask")
 			(remove_unused_layers no)
-			(net 103 "Net-(U10-GND)")
+			(net 106 "Net-(U11-GND)")
 			(pinfunction "GND")
 			(pintype "power_in")
