File: ArduinoBoat/PCBs/TAFLab Boat/TAFLab Sensors.kicad_sch (KiCad schematic)
At the start: 21 parts, among them U1 LM2596S-12

Commit message: PCB edits
Parts:
- removed U2: ~, TAFLab-Footprint-Library:LIS3MDL_Magnometer, symbol TAFLab-Symbol-Library:LISM3DL_Magnometer
- added U2: ~, TAFLab-Footprint-Library:LIS3MDL_Magnometer, symbol TAFLab-Symbol-Library:LIS3MDL_Magnetometer
Connections:
- net at A1.GND1 (GND), U10.3 (GND), U13.6 (GND)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: now also U2.3 (GND); no longer U11.1 (GND), U12.8 (GND), U14.3 (GND), U16.3 (GND), U17.3 (GND)
- net at A1.5V1 (5V), U10.2 (Vin), U11.2 (VCC)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: now also U2.1 (Vin)
- net at A1.SCL, U12.10 (SCL), U13.3 (SCL)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: now also U2.4 (SCL)
- net at A1.SDA, U12.9 (SDA), U13.4 (SDA)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: now also U2.5 (SDA)
- new net: U11.1 (GND), U12.8 (GND), U14.3 (GND), U16.3 (GND), U17.3 (GND)
Changed lines of the file:
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@@
 	)
 	(junction
-		(at 102.87 137.16)
-		(diameter 0)
-		(color 0 0 0 1)
-	)
-	(junction
 		(at 87.63 168.91)
 		(diameter 0)
@@
 	(wire
 		(pts
-			(xy 102.87 137.16) (xy 102.87 100.33)
-		)
-		(stroke
-			(width 0)
-			(type default)
-			(color 0 0 0 1)
-		)
-	)
-	(wire
-		(pts
 			(xy 100.33 167.64) (xy 135.89 167.64)
 		)
@@
 		)
 	)
-	(text_box "NOTES\n\nI2C:\n\n	Inside Boat:\n		- LIS3MDL (Magnetometer)\n		- MPU6050 IMU (Accelerometer)\n		- INA 219 (Battery Power Sensor)\n		- DS3231 (CLK Module)\n\n	Outside Boat:\n		- AS5600 (Magnetic Encoder - Windvane)\n		- BME280 (PHT)\n\nUArt: \n\n	Inside Boat:\n	- GT-U7 (GPS)\n\n	Outside Boat:\n	- Digi Xbee3 (Transmitter/Receiver) \n\nDigital:\n\n	- 45 kg Servo (Rudder)\n	- 45 kg Servo (Sail)\n	- 40A ESC (Propeller)\n	- DS18B20 (Water Temperature Sensor)\n\nAnalog:\n\n	- HW-038 (Water Level Sensor)\n\nSPI:\n\n	- Micro SD Card Read/Write Module\n\nMisc:\n\n	- LM2596S (Voltage Regulator/Detector)"
+	(text_box "NOTES\n\nI2C:\n\n	Inside Boat:\n		- LIS3MDL (Magnetometer)\n		- MPU6050 IMU (Accelerometer)\n		- INA 219 (Battery Power Sensor)\n		- DS3231 (CLK Module)\n\n	Outside Boat:\n		- AS5600 (Magnetic Encoder - Windvane)\n		- BME280 (PHT)\n\nUArt: \n\n	Inside Boat:\n	- GT-U7 (GPS)\n\n	Outside Boat:\n	- Digi Xbee3 (Transmitter/Receiver) \n\nDigital:\n\n	- 45 kg Servo (Rudder)\n	- 45 kg Servo (Sail)\n	- 40A ESC (Propeller)\n	- DS18B20 (Water Temperature Sensor)\n\nAnalog:\n\n	- HW-038 (Water Level Sensor)\n\nSPI:\n\n	- Micro SD Card Read/Write Module\n\nMisc:\n\n	- LM2596S (Voltage Regulator/Detector)\n\nTo-Do:\n- 1 more water level sensor\n- Extra I2C ports\n- On/Off Switch\n- Reset Button\n- LED Indicator\n- Move magnetometer out\n- Wind Speed Sensor"
 		(exclude_from_sim no)
-		(at 15.24 110.49 0)
-		(size 57.15 85.09)
+		(at 13.97 114.3 0)
+		(size 57.15 81.28)
 		(stroke
 			(width 0)
@@
 		(effects
 			(font
-				(size 1.27 1.27)
+				(size 1.016 1.016)
 				(thickness 0.254)
 				(bold yes)
@@
 	)
 	(symbol
-		(lib_id "TAFLab-Symbol-Library:AS5600_Magnetic_Encoder_Windvane")
-		(at 86.36 181.61 0)
+		(lib_id "TAFLab-Symbol-Library:LIS3MDL_Magnetometer")
+		(at 193.04 48.26 90)
 		(unit 1)
 		(exclude_from_sim no)
@@
 		(on_board yes)
 		(dnp no)
-		(property "Reference" "U5"
-			(at 94.742 173.482 0)
+		(fields_autoplaced yes)
+		(property "Reference" "U2"
+			(at 205.74 42.5449 90)
 			(effects
 				(font
 					(size 1.27 1.27)
 				)
+				(justify right)
 			)
 		)
 		(property "Value" "~"
-			(at 93.98 173.99 0)
+			(at 205.74 44.45 90)
 			(effects
 				(font
 					(size 1.27 1.27)
 				)
+				(justify right)
 			)
 		)
-		(property "Footprint" "TAFLab-Footprint-Library:AS5600_Magnetic_Encoder_Windvane"
-			(at 86.36 181.61 0)
+		(property "Footprint" "TAFLab-Footprint-Library:LIS3MDL_Magnometer"
+			(at 193.04 48.26 0)
 			(effects
 				(font
@@
 		)
 		(property "Datasheet" ""
-			(at 86.36 181.61 0)
+			(at 193.04 48.26 0)
 			(effects
 				(font
@@
 		)
 		(property "Description" ""
-			(at 86.36 181.61 0)
+			(at 193.04 48.26 0)
 			(effects
 				(font
@@
 			)
 		)
-		(pin "2"
-		)
-		(pin "7"
-		)
-		(pin "1"
+		(pin "4"
 		)
 		(pin "5"
 		)
-		(pin "4"
-		)
 		(pin "6"
 		)
+		(pin "2"
+		)
 		(pin "3"
 		)
+		(pin "1"
+		)
 		(instances
 			(project "TAFLab Sensors"
 				(path "/596b9502-859d-467d-9cf7-4ff1f1b1dcd6"
-					(reference "U5")
+					(reference "U2")
 					(unit 1)
 				)
@@
 	)
 	(symbol
-		(lib_id "TAFLab-Symbol-Library:LISM3DL_Magnometer")
-		(at 193.04 48.26 90)
+		(lib_id "TAFLab-Symbol-Library:AS5600_Magnetic_Encoder_Windvane")
+		(at 86.36 181.61 0)
 		(unit 1)
 		(exclude_from_sim no)
@@
 		(on_board yes)
 		(dnp no)
-		(fields_autoplaced yes)
-		(property "Reference" "U2"
-			(at 205.74 42.5449 90)
+		(property "Reference" "U5"
+			(at 94.742 173.482 0)
 			(effects
 				(font
 					(size 1.27 1.27)
 				)
-				(justify right)
 			)
 		)
 		(property "Value" "~"
-			(at 205.74 44.45 90)
+			(at 93.98 173.99 0)
 			(effects
 				(font
 					(size 1.27 1.27)
 				)
-				(justify right)
 			)
 		)
-		(property "Footprint" "TAFLab-Footprint-Library:LIS3MDL_Magnometer"
-			(at 193.04 48.26 0)
+		(property "Footprint" "TAFLab-Footprint-Library:AS5600_Magnetic_Encoder_Windvane"
+			(at 86.36 181.61 0)
 			(effects
 				(font
@@
 		)
 		(property "Datasheet" ""
-			(at 193.04 48.26 0)
+			(at 86.36 181.61 0)
 			(effects
 				(font
@@
 		)
 		(property "Description" ""
-			(at 193.04 48.26 0)
+			(at 86.36 181.61 0)
 			(effects
 				(font
@@
 			)
 		)
-		(pin "6"
+		(pin "2"
 		)
-		(pin "5"
+		(pin "7"
 		)
 		(pin "1"
 		)
-		(pin "2"
+		(pin "5"
 		)
 		(pin "4"
 		)
+		(pin "6"
+		)
 		(pin "3"
 		)
@@
 			(project "TAFLab Sensors"
 				(path "/596b9502-859d-467d-9cf7-4ff1f1b1dcd6"
-					(reference "U2")
+					(reference "U5")
 					(unit 1)
 				)
