File: ArduinoBoat/PCBs/TAFLab Controller/TAFLab Controller.kicad_pcb (KiCad board)
At the start: 2 copper layers, 200 x 131 mm, 8 parts

Commit message: Update PCB before review and order w/ Arsh
Other:
- board text added: "BY: NICK BUI"
- board text added: "UC BERKELEY TAFLAB Controller PCB"

Commit message: PCB edits
Parts:
- added R1: 10k, Resistor_SMD:R_0805_2012Metric, F.Cu at (59.1, 35.5)
- added U8: ~, TAFLab-Footprint-Library:PushButton, F.Cu at (63.0, 39.0)
Connections:
- A1 pad 5V4: unconnected-(A1-5V-Pad5V4) -> Net-(D1-A)
- A1 pad GND5: unconnected-(A1-GND-PadGND5) -> Net-(A1-GND-PadGND5)
- A1 pad VIN: unconnected-(A1-PadVIN) -> Net-(U6-VOut)
Routing:
- net Net-(U8-GND): track 0.00 -> 12.1 mm
