File: ArduinoBoat/PCBs/TAFLab Controller/TAFLab Controller.kicad_sch (KiCad schematic)
At the start: 8 parts

Commit message: PCB edits
Parts:
- added D1: LED, LED_THT:LED_D3.0mm_Horizontal_O1.27mm_Z10.0mm, symbol Device:LED
- added R1: 10k, Resistor_SMD:R_0805_2012Metric, symbol Device:R
- added R2: 220, Resistor_SMD:R_0805_2012Metric, symbol Device:R
- added U6: ~, symbol TAFLab-Symbol-Library:PowerSwitch
- added U8: ~, TAFLab-Footprint-Library:PushButton, symbol TAFLab-Symbol-Library:PushButton
Connections:
- net at A1.5V1 (5V), RV1.1, U1.2 (5V)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: now also U8.2 (VCC)
- net at A1.GND1 (GND), RV1.3, U1.1 (GND)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: now also R1.1, U6.3 (GND)
- net at A1.5V4 (5V): now also D1.2 (A)
- net at A1.GND5 (GND): now also R2.1
- net at A1.VIN: now also U6.2 (VOut)
- new net: D1.1 (K), R2.2
- new net: R1.2, U8.1 (GND)
- no-connect marks 3 -> 6
Other:
- note added: "7V Battery"
- note added: "GND"
- note added: "On/Off Switch Vin"
